Commit message: topics i messages comuns a rUBot

File: src/limo_description/urdf/limo.urdf.xacro (robot description, xacro)
@@ -3,4 +3,16 @@
   <xacro:include filename="$(find limo_description)/urdf/limo_xacro.xacro"/>
   <xacro:arg name="use_gz" default="true"/>
+  <xacro:arg name="laser_x" default="0.103"/>
+  <xacro:arg name="laser_y" default="0.0"/>
+  <xacro:arg name="laser_z" default="-0.034"/>
+  <xacro:arg name="laser_roll" default="0.0"/>
+  <xacro:arg name="laser_pitch" default="0.0"/>
+  <xacro:arg name="laser_yaw" default="0.0"/>
+  <xacro:arg name="camera_x" default="0.084"/>
+  <xacro:arg name="camera_y" default="0.0"/>
+  <xacro:arg name="camera_z" default="0.03"/>
+  <xacro:arg name="camera_roll" default="0.0"/>
+  <xacro:arg name="camera_pitch" default="0.0"/>
+  <xacro:arg name="camera_yaw" default="0.0"/>
   <xacro:property name="M_PI" value="3.141592653589793"/>
   <xacro:property name="wheelbase" value="0.20"/>
@@ -47,8 +59,12 @@
   </xacro:limo_wheel>
   <xacro:limo_laser parent_prefix="base_link" frame_prefix="laser">
-    <origin xyz="0.103 0 -0.034" rpy="0 0 0"/>
+    <origin
+      xyz="$(arg laser_x) $(arg laser_y) $(arg laser_z)"
+      rpy="$(arg laser_roll) $(arg laser_pitch) $(arg laser_yaw)"/>
   </xacro:limo_laser>
-  <xacro:limo_depth_camera parent_prefix="base_link" frame_prefix="camera_color">
-    <origin xyz="0.084 0 0.03" rpy="0 0 0"/>
+  <xacro:limo_depth_camera parent_prefix="base_link" frame_prefix="camera">
+    <origin
+      xyz="$(arg camera_x) $(arg camera_y) $(arg camera_z)"
+      rpy="$(arg camera_roll) $(arg camera_pitch) $(arg camera_yaw)"/>
   </xacro:limo_depth_camera>
   <xacro:limo_imu parent_prefix="base_link" frame_prefix="imu">
@@ -66,5 +82,5 @@
         <odom_frame>odom</odom_frame>
         <robot_base_frame>base_footprint</robot_base_frame>
-        <odom_topic>/wheel/odom</odom_topic>
+        <odom_topic>/odom</odom_topic>
         <tf_topic>/tf</tf_topic>
         <odom_publish_frequency>50</odom_publish_frequency>
@@ -76,5 +92,5 @@
       <plugin name="mecanum_controller" filename="libgazebo_ros_planar_move.so">
         <command_topic>/cmd_vel</command_topic>
-        <odometry_topic>/wheel/odom</odometry_topic>
+        <odometry_topic>/odom</odometry_topic>
         <odometry_frame>odom</odometry_frame>
         <odometry_rate>50.0</odometry_rate>
@@ -133,8 +149,8 @@
     </gazebo>
   </xacro:unless>
-  <gazebo reference="camera_color_link">
+  <gazebo reference="camera_link">
     <sensor name="color_camera" type="camera">
       <topic>/camera/color</topic>
-      <gz_frame_id>camera_color_link</gz_frame_id>
+      <gz_frame_id>camera_link</gz_frame_id>
       <always_on>true</always_on>
       <update_rate>15</update_rate>
@@ -158,5 +174,5 @@
           </ros>
           <camera_name>camera_color</camera_name>
-          <frame_name>camera_color_link</frame_name>
+          <frame_name>camera_link</frame_name>
         </plugin>
       </xacro:unless>
